File: kstars-ekos-smd-0-9.kicad_pro/kstars-ekos-smd-0-9.kicad_pro.kicad_sch (KiCad schematic)
At the start: 36 parts, among them J1 Raspberry_Pi_2_3, J2 Conn_01x04, J3 Conn_01x04, U1 AP64501SP-13, U2 TLP3553ATP1_F, U3 TLP3553ATP1_F, U4 TLP3553ATP1_F, U5 TLP3553ATP1_F, U6 TLP241ATP1_F, U7 TLP241ATP1_F

Commit message: Final design submitted to fab.
Connections:
- net GND: now also H5.1; no longer H5.2
- net at U5.4: now also H5.2; no longer H5.1
